Commit message: change files name : op3_description

File: ROBOTIS-OP3-Common/robotis_op3_description/urdf/robotis_op3.structure.leg.xacro (robot description, xacro)
@@ -8,19 +8,19 @@
   <xacro:macro name="robotis_op3_r_leg" params="parent">
   <!-- right hip yaw joint -->
-  <joint name="robotis_op3_r_leg_hip_y" type="revolute">
+  <joint name="r_hip_yaw" type="revolute">
     <axis xyz="0 0 -1" />
     <origin xyz="0.0 -0.035 -0.036" rpy="0 0 0"/>
     <parent link="${parent}"/>
-    <child  link="robotis_op3_r_leg_hip_y_link"/>
-    <limit velocity="6.5" effort="1000" lower="${-pi*0.5}" upper="${pi*0.5}" />
-    <dynamics damping="0.1" friction="0.0" />
-  </joint>
-  <xacro:insert_transmission name="robotis_op3_r_leg_hip_y" />
+    <child  link="r_hip_yaw_link"/>
+    <limit velocity="6.5" effort="1000" lower="${-pi*0.5}" upper="${pi*0.5}" />
+    <dynamics damping="0.1" friction="0.0" />
+  </joint>
+  <xacro:insert_transmission name="r_hip_yaw" />
   <!-- right hip yaw link -->
-  <link name="robotis_op3_r_leg_hip_y_link">
-    <visual>
-      <origin xyz="0 0 0" rpy="0 0 0"/>
-      <geometry>
-        <mesh filename="package://robotis_op3_description/meshes/robotis_op3_r_leg_hip_y_link.stl" scale="0.001 0.001 0.001"/>
+  <link name="r_hip_yaw_link">
+    <visual>
+      <origin xyz="0 0 0" rpy="0 0 0"/>
+      <geometry>
+        <mesh filename="package://robotis_op3_description/meshes/r_hip_yaw_link.stl" scale="0.001 0.001 0.001"/>
       </geometry>
       <material name="grey"/>
@@ -28,19 +28,19 @@
   </link>
   <!-- right hip roll joint -->
-  <joint name="robotis_op3_r_leg_hip_r" type="revolute">
+  <joint name="r_hip_roll" type="revolute">
     <axis xyz="-1 0 0" />
     <origin xyz="-0.021 0.0 -0.0285" rpy="0 0 0"/>
-    <parent link="robotis_op3_r_leg_hip_y_link"/>
-    <child  link="robotis_op3_r_leg_hip_r_link"/>
-    <limit velocity="6.5" effort="1000" lower="${-pi*0.5}" upper="${pi*0.5}" />
-    <dynamics damping="0.1" friction="0.0" />
-  </joint>
-  <xacro:insert_transmission name="robotis_op3_r_leg_hip_r" />
+    <parent link="r_hip_yaw_link"/>
+    <child  link="r_hip_roll_link"/>
+    <limit velocity="6.5" effort="1000" lower="${-pi*0.5}" upper="${pi*0.5}" />
+    <dynamics damping="0.1" friction="0.0" />
+  </joint>
+  <xacro:insert_transmission name="r_hip_roll" />
   <!-- right hip roll link -->
-  <link name="robotis_op3_r_leg_hip_r_link">
-    <visual>
-      <origin xyz="0 0 0" rpy="0 0 0"/>
-      <geometry>
-        <mesh filename="package://robotis_op3_description/meshes/robotis_op3_r_leg_hip_r_link.stl" scale="0.001 0.001 0.001"/>
+  <link name="r_hip_roll_link">
+    <visual>
+      <origin xyz="0 0 0" rpy="0 0 0"/>
+      <geometry>
+        <mesh filename="package://robotis_op3_description/meshes/r_hip_roll_link.stl" scale="0.001 0.001 0.001"/>
       </geometry>
       <material name="grey"/>
@@ -48,19 +48,19 @@
   </link>
   <!-- right hip pitch joint -->
-  <joint name="robotis_op3_r_leg_hip_p" type="revolute">
+  <joint name="r_hip_pitch" type="revolute">
     <axis xyz="0 1 0" />
     <origin xyz="0.0211 0.019 0.0" rpy="0 0 0"/>
-    <parent link="robotis_op3_r_leg_hip_r_link"/>
-    <child  link="robotis_op3_r_leg_hip_p_link"/>
-    <limit velocity="6.5" effort="1000" lower="${-pi*0.5}" upper="${pi*0.5}" />
-    <dynamics damping="0.1" friction="0.0" />
-  </joint>
-  <xacro:insert_transmission name="robotis_op3_r_leg_hip_r" />
+    <parent link="r_hip_roll_link"/>
+    <child  link="r_hip_pitch_link"/>
+    <limit velocity="6.5" effort="1000" lower="${-pi*0.5}" upper="${pi*0.5}" />
+    <dynamics damping="0.1" friction="0.0" />
+  </joint>
+  <xacro:insert_transmission name="r_hip_pitch" />
   <!-- right hip pitch link -->
-  <link name="robotis_op3_r_leg_hip_p_link">
-    <visual>
-      <origin xyz="0 0 0" rpy="0 0 0"/>
-      <geometry>
-        <mesh filename="package://robotis_op3_description/meshes/robotis_op3_r_leg_hip_p_link.stl" scale="0.001 0.001 0.001"/>
+  <link name="r_hip_pitch_link">
+    <visual>
+      <origin xyz="0 0 0" rpy="0 0 0"/>
+      <geometry>
+        <mesh filename="package://robotis_op3_description/meshes/r_hip_pitch_link.stl" scale="0.001 0.001 0.001"/>
       </geometry>
       <material name="grey"/>
@@ -68,19 +68,19 @@
   </link>
   <!-- right knee pitch joint -->
-  <joint name="robotis_op3_r_leg_kn_p" type="revolute">
+  <joint name="r_knee" type="revolute">
     <axis xyz="0 1 0" />
     <origin xyz="0.0 0.0 -0.11" rpy="0 0 0"/>
-    <parent link="robotis_op3_r_leg_hip_p_link"/>
-    <child  link="robotis_op3_r_leg_kn_p_link"/>
-    <limit velocity="6.5" effort="1000" lower="${-pi*0.5}" upper="${pi*0.5}" />
-    <dynamics damping="0.1" friction="0.0" />
-  </joint>
-  <xacro:insert_transmission name="robotis_op3_r_leg_kn_p" />
+    <parent link="r_hip_pitch_link"/>
+    <child  link="r_knee_link"/>
+    <limit velocity="6.5" effort="1000" lower="${-pi*0.5}" upper="${pi*0.5}" />
+    <dynamics damping="0.1" friction="0.0" />
+  </joint>
+  <xacro:insert_transmission name="r_knee" />
   <!-- right knee pitch link -->
-  <link name="robotis_op3_r_leg_kn_p_link">
-    <visual>
-      <origin xyz="0 0 0" rpy="0 0 0"/>
-      <geometry>
-        <mesh filename="package://robotis_op3_description/meshes/robotis_op3_r_leg_kn_p_link.stl" scale="0.001 0.001 0.001"/>
+  <link name="r_knee_link">
+    <visual>
+      <origin xyz="0 0 0" rpy="0 0 0"/>
+      <geometry>
+        <mesh filename="package://robotis_op3_description/meshes/r_knee_link.stl" scale="0.001 0.001 0.001"/>
       </geometry>
       <material name="grey"/>
@@ -88,19 +88,19 @@
   </link>
   <!-- right ankle pitch joint -->
-  <joint name="robotis_op3_r_leg_an_p" type="revolute">
+  <joint name="r_ank_pitch" type="revolute">
     <axis xyz="0 -1 0" />
     <origin xyz="0.0 0.0 -0.11" rpy="0 0 0"/>
-    <parent link="robotis_op3_r_leg_kn_p_link"/>
-    <child  link="robotis_op3_r_leg_an_p_link"/>
-    <limit velocity="6.5" effort="1000" lower="${-pi*0.5}" upper="${pi*0.5}" />
-    <dynamics damping="0.1" friction="0.0" />
-  </joint>
-  <xacro:insert_transmission name="robotis_op3_r_leg_an_p" />
+    <parent link="r_knee_link"/>
+    <child  link="r_ank_pitch_link"/>
+    <limit velocity="6.5" effort="1000" lower="${-pi*0.5}" upper="${pi*0.5}" />
+    <dynamics damping="0.1" friction="0.0" />
+  </joint>
+  <xacro:insert_transmission name="r_ank_pitch" />
   <!-- right ankle pitch link -->
-  <link name="robotis_op3_r_leg_an_p_link">
-    <visual>
-      <origin xyz="0 0 0" rpy="0 0 0"/>
-      <geometry>
-        <mesh filename="package://robotis_op3_description/meshes/robotis_op3_r_leg_an_p_link.stl" scale="0.001 0.001 0.001"/>
+  <link name="r_ank_pitch_link">
+    <visual>
+      <origin xyz="0 0 0" rpy="0 0 0"/>
+      <geometry>
+        <mesh filename="package://robotis_op3_description/meshes/r_ank_pitch_link.stl" scale="0.001 0.001 0.001"/>
       </geometry>
       <material name="grey"/>
@@ -108,19 +108,19 @@
   </link>
   <!-- right ankle roll joint -->
-  <joint name="robotis_op3_r_leg_an_r" type="revolute">
+  <joint name="r_ank_roll" type="revolute">
     <axis xyz="1 0 0" />
     <origin xyz="-0.021 -0.019 0.0" rpy="0 0 0"/>
-    <parent link="robotis_op3_r_leg_an_p_link"/>
-    <child  link="robotis_op3_r_leg_an_r_link"/>
-    <limit velocity="6.5" effort="1000" lower="${-pi*0.5}" upper="${pi*0.5}" />
-    <dynamics damping="0.1" friction="0.0" />
-  </joint>
-  <xacro:insert_transmission name="robotis_op3_r_leg_an_r" />
+    <parent link="r_ank_pitch_link"/>
+    <child  link="r_ank_roll_link"/>
+    <limit velocity="6.5" effort="1000" lower="${-pi*0.5}" upper="${pi*0.5}" />
+    <dynamics damping="0.1" friction="0.0" />
+  </joint>
+  <xacro:insert_transmission name="r_ank_roll" />
   <!-- right ankle roll link -->
-  <link name="robotis_op3_r_leg_an_r_link">
-    <visual>
-      <origin xyz="0 0 0" rpy="0 0 0"/>
-      <geometry>
-        <mesh filename="package://robotis_op3_description/meshes/robotis_op3_r_leg_an_r_link.stl" scale="0.001 0.001 0.001"/>
+  <link name="r_ank_roll_link">
+    <visual>
+      <origin xyz="0 0 0" rpy="0 0 0"/>
+      <geometry>
+        <mesh filename="package://robotis_op3_description/meshes/r_ank_roll_link.stl" scale="0.001 0.001 0.001"/>
       </geometry>
       <material name="grey"/>
@@ -134,19 +134,19 @@
   <xacro:macro name="robotis_op3_l_leg" params="parent">
   <!-- left hip yaw joint -->
-  <joint name="robotis_op3_l_leg_hip_y" type="revolute">
+  <joint name="l_hip_yaw" type="revolute">
     <axis xyz="0 0 -1" />
     <origin xyz="0.0 0.035 -0.036" rpy="0 0 0"/>
     <parent link="${parent}"/>
-    <child  link="robotis_op3_l_leg_hip_y_link"/>
-    <limit velocity="6.5" effort="1000" lower="${-pi*0.5}" upper="${pi*0.5}" />
-    <dynamics damping="0.1" friction="0.0" />
-  </joint>
-  <xacro:insert_transmission name="robotis_op3_l_leg_hip_y" />
+    <child  link="l_hip_yaw_link"/>
+    <limit velocity="6.5" effort="1000" lower="${-pi*0.5}" upper="${pi*0.5}" />
+    <dynamics damping="0.1" friction="0.0" />
+  </joint>
+  <xacro:insert_transmission name="l_hip_yaw" />
   <!-- left hip yaw link -->
-  <link name="robotis_op3_l_leg_hip_y_link">
-    <visual>
-      <origin xyz="0 0 0" rpy="0 0 0"/>
-      <geometry>
-        <mesh filename="package://robotis_op3_description/meshes/robotis_op3_l_leg_hip_y_link.stl" scale="0.001 0.001 0.001"/>
+  <link name="l_hip_yaw_link">
+    <visual>
+      <origin xyz="0 0 0" rpy="0 0 0"/>
+      <geometry>
+        <mesh filename="package://robotis_op3_description/meshes/l_hip_yaw_link.stl" scale="0.001 0.001 0.001"/>
       </geometry>
       <material name="grey"/>
@@ -154,19 +154,19 @@
   </link>
   <!-- left hip roll joint -->
-  <joint name="robotis_op3_l_leg_hip_r" type="revolute">
+  <joint name="l_hip_roll" type="revolute">
     <axis xyz="-1 0 0" />
     <origin xyz="-0.021 0.0 -0.0285" rpy="0 0 0"/>
-    <parent link="robotis_op3_l_leg_hip_y_link"/>
-    <child  link="robotis_op3_l_leg_hip_r_link"/>
-    <limit velocity="6.5" effort="1000" lower="${-pi*0.5}" upper="${pi*0.5}" />
-    <dynamics damping="0.1" friction="0.0" />
-  </joint>
-  <xacro:insert_transmission name="robotis_op3_l_leg_hip_r" />
+    <parent link="l_hip_yaw_link"/>
+    <child  link="l_hip_roll_link"/>
+    <limit velocity="6.5" effort="1000" lower="${-pi*0.5}" upper="${pi*0.5}" />
+    <dynamics damping="0.1" friction="0.0" />
+  </joint>
+  <xacro:insert_transmission name="l_hip_roll" />
   <!-- left hip roll link -->
-  <link name="robotis_op3_l_leg_hip_r_link">
-    <visual>
-      <origin xyz="0 0 0" rpy="0 0 0"/>
-      <geometry>
-        <mesh filename="package://robotis_op3_description/meshes/robotis_op3_l_leg_hip_r_link.stl" scale="0.001 0.001 0.001"/>
+  <link name="l_hip_roll_link">
+    <visual>
+      <origin xyz="0 0 0" rpy="0 0 0"/>
+      <geometry>
+        <mesh filename="package://robotis_op3_description/meshes/l_hip_roll_link.stl" scale="0.001 0.001 0.001"/>
       </geometry>
       <material name="grey"/>
@@ -174,19 +174,19 @@
   </link>
   <!-- left hip pitch joint -->
-  <joint name="robotis_op3_l_leg_hip_p" type="revolute">
+  <joint name="l_hip_pitch" type="revolute">
     <axis xyz="0 -1 0" />
     <origin xyz="0.0211 -0.019 0.0" rpy="0 0 0"/>
-    <parent link="robotis_op3_l_leg_hip_r_link"/>
-    <child  link="robotis_op3_l_leg_hip_p_link"/>
-    <limit velocity="6.5" effort="1000" lower="${-pi*0.5}" upper="${pi*0.5}" />
-    <dynamics damping="0.1" friction="0.0" />
-  </joint>
-  <xacro:insert_transmission name="robotis_op3_l_leg_hip_p" />
+    <parent link="l_hip_roll_link"/>
+    <child  link="l_hip_pitch_link"/>
+    <limit velocity="6.5" effort="1000" lower="${-pi*0.5}" upper="${pi*0.5}" />
+    <dynamics damping="0.1" friction="0.0" />
+  </joint>
+  <xacro:insert_transmission name="l_hip_pitch" />
   <!-- left hip pitch link -->
-  <link name="robotis_op3_l_leg_hip_p_link">
-    <visual>
-      <origin xyz="0 0 0" rpy="0 0 0"/>
-      <geometry>
-        <mesh filename="package://robotis_op3_description/meshes/robotis_op3_l_leg_hip_p_link.stl" scale="0.001 0.001 0.001"/>
+  <link name="l_hip_pitch_link">
+    <visual>
+      <origin xyz="0 0 0" rpy="0 0 0"/>
+      <geometry>
+        <mesh filename="package://robotis_op3_description/meshes/l_hip_pitch_link.stl" scale="0.001 0.001 0.001"/>
       </geometry>
       <material name="grey"/>
@@ -194,19 +194,19 @@
   </link>
   <!-- left knee pitch joint -->
-  <joint name="robotis_op3_l_leg_kn_p" type="revolute">
+  <joint name="l_knee" type="revolute">
     <axis xyz="0 -1 0" />
     <origin xyz="0.0 0.0 -0.11" rpy="0 0 0"/>
-    <parent link="robotis_op3_l_leg_hip_p_link"/>
-    <child  link="robotis_op3_l_leg_kn_p_link"/>
-    <limit velocity="6.5" effort="1000" lower="${-pi*0.5}" upper="${pi*0.5}" />
-    <dynamics damping="0.1" friction="0.0" />
-  </joint>
-  <xacro:insert_transmission name="robotis_op3_l_leg_kn_p" />
+    <parent link="l_hip_pitch_link"/>
+    <child  link="l_knee_link"/>
+    <limit velocity="6.5" effort="1000" lower="${-pi*0.5}" upper="${pi*0.5}" />
+    <dynamics damping="0.1" friction="0.0" />
+  </joint>
+  <xacro:insert_transmission name="l_knee" />
   <!-- left knee pitch link -->
-  <link name="robotis_op3_l_leg_kn_p_link">
-    <visual>
-      <origin xyz="0 0 0" rpy="0 0 0"/>
-      <geometry>
-        <mesh filename="package://robotis_op3_description/meshes/robotis_op3_l_leg_kn_p_link.stl" scale="0.001 0.001 0.001"/>
+  <link name="l_knee_link">
+    <visual>
+      <origin xyz="0 0 0" rpy="0 0 0"/>
+      <geometry>
+        <mesh filename="package://robotis_op3_description/meshes/l_knee_link.stl" scale="0.001 0.001 0.001"/>
       </geometry>
       <material name="grey"/>
@@ -214,19 +214,19 @@
   </link>
   <!-- left ankle pitch joint -->
-  <joint name="robotis_op3_l_leg_an_p" type="revolute">
+  <joint name="l_ank_pitch" type="revolute">
     <axis xyz="0 1 0" />
     <origin xyz="0.0 0.0 -0.11" rpy="0 0 0"/>
-    <parent link="robotis_op3_l_leg_kn_p_link"/>
-    <child  link="robotis_op3_l_leg_an_p_link"/>
-    <limit velocity="6.5" effort="1000" lower="${-pi*0.5}" upper="${pi*0.5}" />
-    <dynamics damping="0.1" friction="0.0" />
-  </joint>
-  <xacro:insert_transmission name="robotis_op3_l_leg_an_p" />
+    <parent link="l_knee_link"/>
+    <child  link="l_ank_pitch_link"/>
+    <limit velocity="6.5" effort="1000" lower="${-pi*0.5}" upper="${pi*0.5}" />
+    <dynamics damping="0.1" friction="0.0" />
+  </joint>
+  <xacro:insert_transmission name="l_ank_pitch" />
   <!-- left ankle pitch link -->
-  <link name="robotis_op3_l_leg_an_p_link">
-    <visual>
-      <origin xyz="0 0 0" rpy="0 0 0"/>
-      <geometry>
-        <mesh filename="package://robotis_op3_description/meshes/robotis_op3_l_leg_an_p_link.stl" scale="0.001 0.001 0.001"/>
+  <link name="l_ank_pitch_link">
+    <visual>
+      <origin xyz="0 0 0" rpy="0 0 0"/>
+      <geometry>
+        <mesh filename="package://robotis_op3_description/meshes/l_ank_pitch_link.stl" scale="0.001 0.001 0.001"/>
       </geometry>
       <material name="grey"/>
@@ -234,19 +234,19 @@
   </link>
   <!-- left ankle roll joint -->
-  <joint name="robotis_op3_l_leg_an_r" type="revolute">
+  <joint name="l_ank_roll" type="revolute">
     <axis xyz="1 0 0" />
     <origin xyz="-0.021 0.019 0.0" rpy="0 0 0"/>
-    <parent link="robotis_op3_l_leg_an_p_link"/>
-    <child  link="robotis_op3_l_leg_an_r_link"/>
-    <limit velocity="6.5" effort="1000" lower="${-pi*0.5}" upper="${pi*0.5}" />
-    <dynamics damping="0.1" friction="0.0" />
-  </joint>
-  <xacro:insert_transmission name="robotis_op3_l_leg_an_r" />
+    <parent link="l_ank_pitch_link"/>
+    <child  link="l_ank_roll_link"/>
+    <limit velocity="6.5" effort="1000" lower="${-pi*0.5}" upper="${pi*0.5}" />
+    <dynamics damping="0.1" friction="0.0" />
+  </joint>
+  <xacro:insert_transmission name="l_ank_roll" />
   <!-- left ankle roll link -->
-  <link name="robotis_op3_l_leg_an_r_link">
-    <visual>
-      <origin xyz="0 0 0" rpy="0 0 0"/>
-      <geometry>
-        <mesh filename="package://robotis_op3_description/meshes/robotis_op3_l_leg_an_r_link.stl" scale="0.001 0.001 0.001"/>
+  <link name="l_ank_roll_link">
+    <visual>
+      <origin xyz="0 0 0" rpy="0 0 0"/>
+      <geometry>
+        <mesh filename="package://robotis_op3_description/meshes/l_ank_roll_link.stl" scale="0.001 0.001 0.001"/>
       </geometry>
       <material name="grey"/>

File: ROBOTIS-OP3-Common/robotis_op3_description/urdf/robotis_op3.xacro (robot description, xacro)
@@ -29,5 +29,5 @@
       <origin xyz="0 0 0" rpy="0 0 0"/>
       <geometry>
-        <mesh filename="package://robotis_op3_description/meshes/robotis_op3_body_link.stl" scale="0.001 0.001 0.001"/>
+        <mesh filename="package://robotis_op3_description/meshes/body_link.stl" scale="0.001 0.001 0.001"/>
       </geometry>
       <material name="grey"/>

Commit message: change robotis_op3 urdf change camera package change soccer_demo : add callbackThread

File: ROBOTIS-OP3-Common/robotis_op3_description/urdf/robotis_op3.structure.arm.xacro (robot description, xacro)
@@ -10,5 +10,5 @@
   <joint name="r_sho_pitch" type="revolute">
     <axis xyz="0 -1 0" />
-    <origin xyz="0.0 -0.062 0.07" rpy="0 0 0"/>
+    <origin xyz="-0.001 -0.06 0.07" rpy="0 0 0"/>
     <parent link="${parent}"/>
     <child link="r_sho_pitch_link"/>
@@ -29,6 +29,6 @@
   <!-- right shoulder roll joint -->
   <joint name="r_sho_roll" type="revolute">
-    <axis xyz="1 0 0" />
-    <origin xyz="0.019 -0.019 -0.0465" rpy="0 0 0"/>
+    <axis xyz="-1 0 0" />
+    <origin xyz="0.019 -0.0285 0.0" rpy="0 0 0"/>
     <parent link="r_sho_pitch_link"/>
     <child link="r_sho_roll_link"/>
@@ -50,5 +50,5 @@
   <joint name="r_el" type="revolute">
     <axis xyz="1 0 0" />
-    <origin xyz="0.0 -0.09025 0" rpy="0 0 0"/>
+    <origin xyz="0.0 -0.0905 0" rpy="0 0 0"/>
     <parent link="r_sho_roll_link"/>
     <child link="r_el_link"/>
@@ -76,5 +76,5 @@
   <joint name="l_sho_pitch" type="revolute">
     <axis xyz="0 1 0" />
-    <origin xyz="0.0 0.062 0.07" rpy="0 0 0"/>
+    <origin xyz="-0.001 0.06 0.07" rpy="0 0 0"/>
     <parent link="${parent}"/>
     <child link="l_sho_pitch_link"/>
@@ -95,6 +95,6 @@
   <!-- left shoulder roll joint -->
   <joint name="l_sho_roll" type="revolute">
-    <axis xyz="1 0 0" />
-    <origin xyz="0.019 0.019 -0.0465" rpy="0 0 0"/>
+    <axis xyz="-1 0 0" />
+    <origin xyz="0.019 0.0285 0.0" rpy="0 0 0"/>
     <parent link="l_sho_pitch_link"/>
     <child link="l_sho_roll_link"/>
@@ -116,5 +116,5 @@
   <joint name="l_el" type="revolute">
     <axis xyz="1 0 0" />
-    <origin xyz="0.0 0.09025 0" rpy="0 0 0"/>
+    <origin xyz="0.0 0.0905 0" rpy="0 0 0"/>
     <parent link="l_sho_roll_link"/>
     <child link="l_el_link"/>

File: ROBOTIS-OP3-Common/robotis_op3_description/urdf/robotis_op3.structure.head.xacro (robot description, xacro)
@@ -26,5 +26,5 @@
   <!-- head pitch joint -->
   <joint name="head_tilt" type="revolute">
-    <axis xyz="0 1 0" />
+    <axis xyz="0 -1 0" />
     <origin xyz="0.0255 -0.019 0.03725" rpy="0 0 0"/>
     <parent link="head_pan_link"/>
@@ -46,5 +46,5 @@
   <!-- camera joint -->
   <joint name="cam" type="fixed">
-    <origin xyz="0.017 0.019 0.0385" rpy="${-pi*0.5} 0 ${-pi*0.5}"/>
+    <origin xyz="0.025 0.019 0.038" rpy="${-pi*0.5} 0 ${-pi*0.5}"/>
     <parent link="head_tilt_link"/>
     <child link="cam_link"/>
