Commit message: model change

File: ROBOTIS-OP3-Common/robotis_op3_description/urdf/robotis_op3.structure.head.xacro (robot description, xacro)
@@ -1,14 +1,14 @@
-<?xml version="1.0"?>
+<?xml version="1.0" ?>
 <robot xmlns:xacro="http://ros.org/wiki/xacro">
   <xacro:property name="pi" value="3.141592654" />
-  <!-- robotis_op3 head -->
+  <!-- head -->
   <xacro:macro name="robotis_op3_head" params="parent">
   <!-- head yaw joint -->
   <joint name="head_pan" type="revolute">
+    <parent link="${parent}"/>
+    <child link="head_pan_link"/>
+    <origin xyz="-0.001 0.0 0.1365" rpy="0 0 0" />
     <axis xyz="0 0 1" />
-    <origin xyz="0.0 0.0 0.102" rpy="0 0 0"/>
-    <parent link="${parent}"/>
-    <child  link="head_pan_link"/>
-    <limit velocity="6.5" effort="1000" lower="${-pi*0.5}" upper="${pi*0.5}" />
+    <limit effort="1000" velocity="100" lower="${-pi*0.6}" upper="${pi*0.6}" />
     <dynamics damping="0.1" friction="0.0" />
   </joint>
@@ -17,34 +17,38 @@
   <link name="head_pan_link">
     <visual>
-      <origin xyz="0 0 0" rpy="0 0 0"/>
-      <geometry>
-        <mesh filename="package://robotis_op3_description/meshes/head_pan_link.stl" scale="0.001 0.001 0.001"/>
-      </geometry>
-      <material name="grey"/>
+      <xacro:insert_mesh_head_pan_link />
     </visual>
+    <collision>
+      <xacro:insert_mesh_head_pan_link />
+    </collision>
+    <inertial>
+      <xacro:insert_inertia_head_pan_link />
+    </inertial>
   </link>
   <!-- head pitch joint -->
   <joint name="head_tilt" type="revolute">
+    <parent link="head_pan_link"/>
+    <child link="head_tilt_link"/>
+    <origin xyz="0.010 0.019 0.0285" rpy="0 0 0" />
     <axis xyz="0 -1 0" />
-    <origin xyz="0.0255 -0.019 0.03725" rpy="0 0 0"/>
-    <parent link="head_pan_link"/>
-    <child  link="head_tilt_link"/>
-    <limit velocity="6.5" effort="1000" lower="${-pi*0.5}" upper="${pi*0.5}" />
+    <limit effort="1000" velocity="100" lower="${-pi*0.6}" upper="${pi*0.6}" />
     <dynamics damping="0.1" friction="0.0" />
   </joint>
   <xacro:insert_transmission name="head_tilt" />
-  <!-- head pitch link -->
+  <!-- head yaw link -->
   <link name="head_tilt_link">
     <visual>
-      <origin xyz="0 0 0" rpy="0 0 0"/>
-      <geometry>
-        <mesh filename="package://robotis_op3_description/meshes/head_tilt_link.stl" scale="0.001 0.001 0.001"/>
-      </geometry>
-      <material name="grey"/>
+      <xacro:insert_mesh_head_tilt_link />
     </visual>
+    <collision>
+      <xacro:insert_mesh_head_tilt_link />
+    </collision>
+    <inertial>
+      <xacro:insert_inertia_head_tilt_link />
+    </inertial>
   </link>
   <!-- camera joint -->
   <joint name="cam" type="fixed">
-    <origin xyz="0.025 0.019 0.038" rpy="${-pi*0.5} 0 ${-pi*0.5}"/>
+    <origin xyz="0.01425 -0.019 0.04975" rpy="${-pi*0.5} 0 ${-pi*0.5}"/>
     <parent link="head_tilt_link"/>
     <child link="cam_link"/>

File: ROBOTIS-OP3-Common/robotis_op3_description/urdf/robotis_op3.transmissions.xacro (robot description, xacro)
@@ -1,15 +1,15 @@
 <?xml version="1.0"?>
 <robot xmlns:xacro="http://ros.org/wiki/xacro">
-	<xacro:macro name="insert_transmission" params="name">
-		<transmission name="${name}_tran">
-			<type>transmission_interface/SimpleTransmission</type>
-			<joint name="${name}">
-				<hardwareInterface>EffortJointInterface</hardwareInterface>
-			</joint>
-			<actuator name="${name}_motor">
-				<hardwareInterface>EffortJointInterface</hardwareInterface>
-				<mechanicalReduction>1</mechanicalReduction>
-			</actuator>
-		</transmission>
-	</xacro:macro>
+  <xacro:macro name="insert_transmission" params="name">
+    <transmission name="${name}_tran">
+      <type>transmission_interface/SimpleTransmission</type>
+      <joint name="${name}">
+        <hardwareInterface>EffortJointInterface</hardwareInterface>
+      </joint>
+      <actuator name="${name}_motor">
+        <hardwareInterface>EffortJointInterface</hardwareInterface>
+        <mechanicalReduction>1</mechanicalReduction>
+      </actuator>
+    </transmission>
+  </xacro:macro>
 </robot>
